File: HW/CO2_stm_sensor/wakeup_circuit.kicad_sch (KiCad schematic)
At the start: 14 parts, among them SW2 USER_WAKEUP

Commit message: hw v1.0
Parts:
- removed CMU_SWITCH-Active_High1, WAKE_UP_SWITCH-Active_Low1: TPS22917DBVR, SOT95P280X145-6N, symbol TPS22917DBVR:TPS22917DBVR
- removed SW2: USER_WAKEUP, symbol Switch:SW_MEC_5G
- added IC2, IC3: SWITCH_TPS22917DBVR, JLC:SOT95P280X145-6N, symbol STM32_CO2:SWITCH_TPS22917DBVR
- added S1: USR_WAKEUP, JLC:pushbutton_EVQPUC02K, symbol CustomSymbols:pushbutton
- added TP1, TP3, TP4: TestPoint, Connector_PinHeader_2.54mm:PinHeader_1x01_P2.54mm_Vertical, symbol Connector:TestPoint
- C16, C17, C18, C19, C20: footprint (none) -> Capacitor_SMD:C_0805_2012Metric_Pad1.18x1.45mm_HandSolder
- R10, R11, R12, R13, R14: footprint (none) -> Resistor_SMD:R_0805_2012Metric
Connections:
- net BATTERY_PWR: now also IC2.1 (VIN), IC3.1 (VIN)
- net GND: now also IC2.2 (GND), IC3.2 (GND), S1.3
- net MCU_PWR: now also IC2.6 (VOUT), IC3.6 (VOUT), TP4.1
- net MCU_PWR_ON: now also IC3.3 (ON), TP3.1
- net RTC_INT: now also IC2.3 (ON), S1.1, TP1.1
- net at C16.2: now also IC2.4 (CT)
- net at R10.1: now also IC2.5 (QOD)
- net at R14.1: now also IC3.5 (QOD)
- net at C18.2: now also IC3.4 (CT)
- no-connect marks 1 -> 3
