File: HW/CO2_stm_sensor/CO2_stm_sensor.kicad_pcb (KiCad board)
At the start: 2 copper layers, 35 x 92 mm, 71 parts, among them IC1 SCD41-D-R2, IC2 SWITCH_TPS22917DBVR, IC3 SWITCH_TPS22917DBVR, J1 Conn_1x4, J2 Conn_1x4, J3 Conn_1x6, J4 Conn_1x6, U2 P_MOSFET_AO3407A, U3 USBC_16PIN, U4 ESC_Protection_USBLC6-2SC6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

Commit message: FIRST ORDER git statusgit status
Parts:
- moved R15 4.34 mm to (128.5, 103.2), turned to -90 degrees
- moved R16 4.00 mm to (128.5, 95.8), turned to -90 degrees
- moved D2 3.50 mm to (128.5, 107.0), turned to 90 degrees
- moved D3 3.50 mm to (128.5, 99.5), turned to 90 degrees
Routing:
- net Net-(U5-PB0): track 23.7 -> 18.2 mm
- net GND: track 37.7 -> 33.9 mm, vias 87 -> 86
- net Net-(D3-A): track 1.56 -> 3.38 mm
- net Net-(U5-PA3): track 10.6 -> 12.0 mm

Commit message: LDO GND connected and pwr led rotated in the pcb design
Parts:
- R1: value 2k R -> 5k R
- moved R1 4.33 mm to (128.5, 113.1), turned to -90 degrees
- moved D1 3.78 mm to (128.5, 116.8), turned to 90 degrees
Connections:
- LDO1 pad 1: unconnected-(LDO1-ADJ(GND)-Pad1) -> GND
Routing:
- net Net-(LDO1-VIN): track 43.7 -> 48.4 mm
- net GND: track 33.9 -> 38.4 mm, vias 86 -> 87
- net Net-(D1-A): track 2.49 -> 1.75 mm
